File: RFM12B-V1.1.brd (EAGLE design)
At the start: 19.2 x 28.2 mm, 13 parts, among them J1 NRF connector, J2 SD card

Commit message: Version sent to OSH
Latest revision sent to PCB fab
Parts:
- removed R2: 1K, resistor:M0805
- added R11: 1K, resistor:M0805
- added R13: 100, resistor:M0805
- moved LED2 0.13 mm to (1.40, 2.67)
- renumbered C1 to C10, C2 to C11, R1 to R10, R3 to R12
Connections:
- new net N$6: R13.2, U$2.FFS
- net CE: now also R13.1
- net N$3: now also R11.1; no longer R2.1
- net VCC: now also R11.2; no longer R2.2
Routing:
- net CE: track 22.3 -> 68.2 mm
- net N$6: track 0.00 -> 35.9 mm
- net VCC: track 89.9 -> 68.5 mm
Other:
- board text added: "OOK"
- board text added: "http://hallard.me V1.1"
